File: kicad_files/Knobert_MacroPad.kicad_sch (KiCad schematic)
At the start: 0 parts

Commit message: Added schematic
Other:
- added sheet LedMatrix (ledmatrix.kicad_sch)
- added sheet MCU (mcu.kicad_sch)
- added sheet Miscellaneous (miscellaneous.kicad_sch)
- added sheet SwitchMatrix (switchmatrix.kicad_sch)
Changed lines of the file:
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@@
-(kicad_sch (version 20210621) (generator eeschema)
+(kicad_sch (version 20221206) (generator eeschema)
   (paper "A4")
+  (sheet (at 19.05 19.05) (size 25.4 19.05) (fields_autoplaced)
+    (stroke (width 0.1524) (type solid))
+    (fill (color 0 0 0 0.0000))
+    (property "Sheetname" "MCU" (at 19.05 18.3384 0)
+      (effects (font (size 1.27 1.27)) (justify left bottom))
+    )
+    (property "Sheetfile" "mcu.kicad_sch" (at 19.05 38.6846 0)
+      (effects (font (size 1.27 1.27)) (justify left top))
+    )
+    (instances
+      (project "Knobert_MacroPad"
+        (path "/9ce6b20d-0a6c-402a-b232-5eafd6242eb3" (page "2"))
+      )
+    )
+  )
+  (sheet (at 114.3 19.05) (size 25.4 19.05) (fields_autoplaced)
+    (stroke (width 0.1524) (type solid))
+    (fill (color 0 0 0 0.0000))
+    (property "Sheetname" "Miscellaneous" (at 114.3 18.3384 0)
+      (effects (font (size 1.27 1.27)) (justify left bottom))
+    )
+    (property "Sheetfile" "miscellaneous.kicad_sch" (at 114.3 38.6846 0)
+      (effects (font (size 1.27 1.27)) (justify left top))
+    )
+    (instances
+      (project "Knobert_MacroPad"
+        (path "/9ce6b20d-0a6c-402a-b232-5eafd6242eb3" (page "5"))
+      )
+    )
+  )
+  (sheet (at 82.55 19.05) (size 25.4 19.05) (fields_autoplaced)
+    (stroke (width 0.1524) (type solid))
+    (fill (color 0 0 0 0.0000))
+    (property "Sheetname" "LedMatrix" (at 82.55 18.3384 0)
+      (effects (font (size 1.27 1.27)) (justify left bottom))
+    )
+    (property "Sheetfile" "ledmatrix.kicad_sch" (at 82.55 38.6846 0)
+      (effects (font (size 1.27 1.27)) (justify left top))
+    )
+    (instances
+      (project "Knobert_MacroPad"
+        (path "/9ce6b20d-0a6c-402a-b232-5eafd6242eb3" (page "4"))
+      )
+    )
+  )
+  (sheet (at 50.8 19.05) (size 25.4 19.05) (fields_autoplaced)
+    (stroke (width 0.1524) (type solid))
+    (fill (color 0 0 0 0.0000))
+    (property "Sheetname" "SwitchMatrix" (at 50.8 18.3384 0)
+      (effects (font (size 1.27 1.27)) (justify left bottom))
+    )
+    (property "Sheetfile" "switchmatrix.kicad_sch" (at 50.8 38.6846 0)
+      (effects (font (size 1.27 1.27)) (justify left top))
+    )
+    (instances
+      (project "Knobert_MacroPad"
+        (path "/9ce6b20d-0a6c-402a-b232-5eafd6242eb3" (page "3"))
+      )
+    )
+  )
   (sheet_instances
     (path "/" (page "1"))
