File: kicad_files/Knobert_MacroPad.kicad_pcb (KiCad board)
At the start: 2 copper layers, 0 parts

Commit message: beta pcb layout
Parts:
- added C1: locked, Capacitor_SMD:C_0805_2012Metric, B.Cu at (43.8, 162.1)
- added C10: 100n, Capacitor_SMD:C_0805_2012Metric, B.Cu at (72.6, 170.6)
- added C11: 100n, Capacitor_SMD:C_0805_2012Metric, B.Cu at (72.6, 189.7)
- added C12: 100n, Capacitor_SMD:C_0805_2012Metric, B.Cu at (91.7, 151.6)
- added C13: 100n, Capacitor_SMD:C_0805_2012Metric, B.Cu at (91.7, 170.6)
- added C14: 100n, Capacitor_SMD:C_0805_2012Metric, B.Cu at (91.7, 189.7)
- added C15: 100n, Capacitor_SMD:C_0805_2012Metric, B.Cu at (110.7, 151.6)
- added C16: 100n, Capacitor_SMD:C_0805_2012Metric, B.Cu at (110.7, 170.6)
- added C17: 100n, Capacitor_SMD:C_0805_2012Metric, B.Cu at (110.7, 189.7)
- added C18: 100n, Capacitor_SMD:C_0805_2012Metric, B.Cu at (129.8, 151.6)
- added C19: 100n, Capacitor_SMD:C_0805_2012Metric, B.Cu at (129.8, 170.6)
- added C2: 10n, Capacitor_SMD:C_0805_2012Metric, B.Cu at (43.8, 164.3)
- added C20: 100n, Capacitor_SMD:C_0805_2012Metric, B.Cu at (129.8, 189.7)
- added C21: 10n, Capacitor_SMD:C_0805_2012Metric, B.Cu at (50.0, 159.0)
- added C22: 10n, Capacitor_SMD:C_0805_2012Metric, B.Cu at (41.3, 159.0)
- added C23: 1u, Capacitor_SMD:C_0805_2012Metric, B.Cu at (56.4, 160.8)
- added C24: 1u, Capacitor_SMD:C_0805_2012Metric, B.Cu at (52.3, 169.2)
- added C25: 100n, Capacitor_SMD:C_0805_2012Metric, F.Cu at (48.9, 183.1)
- added C26: 10u, Capacitor_SMD:C_0805_2012Metric, F.Cu at (49.3, 172.5)
- added C3: 100n, Capacitor_SMD:C_0805_2012Metric, B.Cu at (36.8, 167.6)
- added C4: 100n, Capacitor_SMD:C_0805_2012Metric, B.Cu at (36.8, 175.8)
- added C5: 100n, Capacitor_SMD:C_0805_2012Metric, B.Cu at (43.8, 178.6)
- added C6: 4.7u, Capacitor_SMD:C_0805_2012Metric, B.Cu at (43.8, 180.6)
- added C7: 100n, Capacitor_SMD:C_0805_2012Metric, B.Cu at (52.7, 174.7)
- added C8: 4.7u, Capacitor_SMD:C_0805_2012Metric, B.Cu at (51.1, 173.1)
- added C9: 100n, Capacitor_SMD:C_0805_2012Metric, B.Cu at (72.6, 151.6)
- added D1: 1N4148W, acheron_Components:D_SOD-123, B.Cu at (59.5, 150.0)
- added D10: 1N4148W, acheron_Components:D_SOD-123, B.Cu at (116.7, 150.0)
- added D11: 1N4148W, acheron_Components:D_SOD-123, B.Cu at (116.7, 169.1)
- added D12: 1N4148W, acheron_Components:D_SOD-123, B.Cu at (116.7, 188.1)
- added D13: 1N4148W, acheron_Components:D_SOD-123, B.Cu at (53.6, 155.4)
- added D14: SK6812MINI-E, acheron_Components:SK6812MINI_3535_6028_3.2x2.8mm_Round, B.Cu at (67.9, 152.4)
- added D15: SK6812MINI-E, acheron_Components:SK6812MINI_3535_6028_3.2x2.8mm_Round, B.Cu at (67.9, 171.4)
- added D16: SK6812MINI-E, acheron_Components:SK6812MINI_3535_6028_3.2x2.8mm_Round, B.Cu at (67.9, 190.5)
- added D17: SK6812MINI-E, acheron_Components:SK6812MINI_3535_6028_3.2x2.8mm_Round, B.Cu at (86.9, 152.4)
- added D18: SK6812MINI-E, acheron_Components:SK6812MINI_3535_6028_3.2x2.8mm_Round, B.Cu at (86.9, 171.4)
- added D19: SK6812MINI-E, acheron_Components:SK6812MINI_3535_6028_3.2x2.8mm_Round, B.Cu at (86.9, 190.5)
- added D2: 1N4148W, acheron_Components:D_SOD-123, B.Cu at (59.5, 169.1)
- added D20: SK6812MINI-E, acheron_Components:SK6812MINI_3535_6028_3.2x2.8mm_Round, B.Cu at (106.0, 152.4)
- added D21: SK6812MINI-E, acheron_Components:SK6812MINI_3535_6028_3.2x2.8mm_Round, B.Cu at (106.0, 171.4)
- added D22: SK6812MINI-E, acheron_Components:SK6812MINI_3535_6028_3.2x2.8mm_Round, B.Cu at (106.0, 190.5)
- added D23: SK6812MINI-E, acheron_Components:SK6812MINI_3535_6028_3.2x2.8mm_Round, B.Cu at (125.0, 152.4)
- added D24: SK6812MINI-E, acheron_Components:SK6812MINI_3535_6028_3.2x2.8mm_Round, B.Cu at (125.0, 171.4)
- added D25: SK6812MINI-E, acheron_Components:SK6812MINI_3535_6028_3.2x2.8mm_Round, B.Cu at (125.0, 190.5)
- added D26: RB060M-60TR, acheron_Components:D_SOD-123, B.Cu at (52.1, 164.6)
- added D27: 1N4148W, acheron_Components:D_SOD-123, F.Cu at (42.6, 177.9)
- added D3: 1N4148W, acheron_Components:D_SOD-123, B.Cu at (59.5, 188.1)
- added D4: 1N4148W, acheron_Components:D_SOD-123, B.Cu at (78.6, 150.0)
- added D5: 1N4148W, acheron_Components:D_SOD-123, B.Cu at (78.6, 169.1)
- added D6: 1N4148W, acheron_Components:D_SOD-123, B.Cu at (78.6, 188.1)
- added D7: 1N4148W, acheron_Components:D_SOD-123, B.Cu at (97.6, 150.0)
- added D8: 1N4148W, acheron_Components:D_SOD-123, B.Cu at (97.6, 169.1)
- added D9: 1N4148W, acheron_Components:D_SOD-123, B.Cu at (97.6, 188.1)
- added F1: mSMD110-16V, acheron_Components:Fuse_1812_4532, B.Cu at (58.2, 156.5)
- added H1: MountingHole, acheron_MountingHoles:MountingHole_2.5x4.0mm, F.Cu at (77.4, 156.0)
- added H2: MountingHole, acheron_MountingHoles:MountingHole_2.5x4.0mm, F.Cu at (115.5, 156.0)
- added H3: MountingHole, acheron_MountingHoles:MountingHole_2.5x4.0mm, F.Cu at (115.5, 175.0)
- added H4: MountingHole, acheron_MountingHoles:MountingHole_2.5x4.0mm, F.Cu at (58.3, 175.0)
- added H5: MountingHole, acheron_Hardware:MouseBite_IPC7351, F.Cu at (57.9, 135.1)
- added H6: MountingHole, acheron_Hardware:MouseBite_IPC7351, F.Cu at (52.9, 135.1)
- added H9: MountingHole, acheron_Graphics:OSH_Logo_22.5x8.5mm, F.Cu at (47.2, 161.8)
- added J1: ARM JTAG, acheron_Connectors:PinHeader_2x5_P2.54mm_Vertical_Staggered, F.Cu at (-112.8, 161.5)
- added J3: Conn_01x04, acheron_Connectors:SM04B-SRSS-TB(LF)(SN)_mounting-reliefs, B.Cu at (53.3, 182.9)
- added J4: Oled, acheron_Connectors:PinHeader_1x4_P2.54mm_Vertical, F.Cu at (45.6, 191.8)
- added L1: L_Ferrite, Inductor_SMD:L_1206_3216Metric_Pad1.42x1.75mm_HandSolder, B.Cu at (63.8, 137.8)
- added L2: L_Ferrite, Inductor_SMD:L_1206_3216Metric_Pad1.42x1.75mm_HandSolder, B.Cu at (38.9, 139.2)
- added Q1: DTC123JKAT146, Package_TO_SOT_SMD:SOT-23, F.Cu at (41.7, 182.4)
- added R1: 4.7k, Resistor_SMD:R_0805_2012Metric, B.Cu at (42.0, 188.6)
- added R10: 100R, Resistor_SMD:R_0805_2012Metric, B.Cu at (112.8, 170.6)
- added R11: 100R, Resistor_SMD:R_0805_2012Metric, B.Cu at (112.8, 189.7)
- added R12: 100R, Resistor_SMD:R_0805_2012Metric, B.Cu at (131.8, 151.6)
- added R13: 100R, Resistor_SMD:R_0805_2012Metric, B.Cu at (131.8, 170.6)
- added R14: 100R, Resistor_SMD:R_0805_2012Metric, B.Cu at (131.8, 189.7)
- added R15: 10k, Resistor_SMD:R_0805_2012Metric, B.Cu at (47.0, 157.7)
- added R16: 10k, Resistor_SMD:R_0805_2012Metric, B.Cu at (44.2, 157.7)
- added R17: 10k, Resistor_SMD:R_0805_2012Metric, B.Cu at (50.0, 157.0)
- added R18: 10k, Resistor_SMD:R_0805_2012Metric, B.Cu at (41.3, 157.0)
- added R19: 5.1k, Resistor_SMD:R_0805_2012Metric, B.Cu at (52.8, 142.2)
- added R2: 4.7k, Resistor_SMD:R_0805_2012Metric, B.Cu at (45.1, 188.6)
- added R20: 5.1k, Resistor_SMD:R_0805_2012Metric, B.Cu at (57.9, 142.2)
- added R21: 100k, Resistor_SMD:R_0805_2012Metric, B.Cu at (56.4, 163.3)
- added R22: 100k, Resistor_SMD:R_0805_2012Metric, B.Cu at (55.4, 169.9)
- added R23: 330k, Resistor_SMD:R_0805_2012Metric, F.Cu at (43.0, 173.2)
- added R24: 1M, Resistor_SMD:R_0805_2012Metric, F.Cu at (45.8, 172.5)
- added R25: 100R, Resistor_SMD:R_0805_2012Metric, F.Cu at (45.3, 183.1)
- added R3: 100R, Resistor_SMD:R_0805_2012Metric, B.Cu at (74.7, 151.6)
- added R4: 100R, Resistor_SMD:R_0805_2012Metric, B.Cu at (74.7, 170.6)
- added R5: 100R, Resistor_SMD:R_0805_2012Metric, B.Cu at (74.7, 189.7)
- added R6: 100R, Resistor_SMD:R_0805_2012Metric, B.Cu at (93.7, 151.6)
- added R7: 100R, Resistor_SMD:R_0805_2012Metric, B.Cu at (93.7, 170.6)
- added R8: 100R, Resistor_SMD:R_0805_2012Metric, B.Cu at (93.7, 189.7)
- added R9: 100R, Resistor_SMD:R_0805_2012Metric, B.Cu at (112.8, 151.6)
- added SW1: Mechanical_Switch, acheron_MXH:MX100H, B.Cu at (67.9, 146.4)
- added SW10: Mechanical_Switch, acheron_MXH:MX100H, B.Cu at (125.0, 146.4)
- added SW11: Mechanical_Switch, acheron_MXH:MX100H, B.Cu at (125.0, 165.5)
- added SW12: Mechanical_Switch, acheron_MXH:MX100H, B.Cu at (125.0, 184.5)
- added SW13: EC11, acheron_Hardware:ALPS_EC11E, B.Cu at (45.6, 146.5)
- added SW14: SW_SPST, acheron_Hardware:K2-1187SQ-A4SW-06, F.Cu at (47.1, 177.8)
- added SW2: Mechanical_Switch, acheron_MXH:MX100H, B.Cu at (67.9, 165.5)
- added SW3: Mechanical_Switch, acheron_MXH:MX100H, B.Cu at (67.9, 184.5)
- added SW4: Mechanical_Switch, acheron_MXH:MX100H, B.Cu at (86.9, 146.4)
- added SW5: Mechanical_Switch, acheron_MXH:MX100H, B.Cu at (86.9, 165.5)
- added SW6: Mechanical_Switch, acheron_MXH:MX100H, B.Cu at (86.9, 184.5)
- added SW7: Mechanical_Switch, acheron_MXH:MX100H, B.Cu at (106.0, 146.4)
- added SW8: Mechanical_Switch, acheron_MXH:MX100H, B.Cu at (106.0, 165.5)
- added SW9: Mechanical_Switch, acheron_MXH:MX100H, B.Cu at (106.0, 184.5)
- added U1: STM32F072-LQFP48, acheron_Components:LQFP-48_7x7mm_P0.5mm, B.Cu at (43.7, 171.5)
- added U2: USBLC6-2SC6, acheron_Components:SOT-23-6, B.Cu at (55.5, 149.6)
- added U3: MCP1700-3302E, Package_TO_SOT_SMD:SOT-23, B.Cu at (55.4, 166.6)
- added locked: locked, acheron_Connectors:USB_C_Receptacle_Hroparts_TYPE-C-31-M-12, B.Cu at (55.4, 138.4)
Routing:
- net 5V: track 0.00 -> 296.5 mm, vias 0 -> 6
- net C3: track 0.00 -> 176.4 mm, vias 0 -> 5
- net C2: track 0.00 -> 147.4 mm, vias 0 -> 6
- net R0: track 0.00 -> 105.9 mm, vias 0 -> 6
- net R2: track 0.00 -> 102.6 mm, vias 0 -> 8
- net R1: track 0.00 -> 97.0 mm, vias 0 -> 8
- net C1: track 0.00 -> 94.6 mm, vias 0 -> 6
- net 3V3: track 0.00 -> 89.3 mm, vias 0 -> 3
- net Net-(D15-DIN): track 0.00 -> 89.0 mm
- net Net-(D16-DIN): track 0.00 -> 89.0 mm
- net C0: track 0.00 -> 76.2 mm, vias 0 -> 4
- net D+: track 0.00 -> 42.2 mm, vias 0 -> 2
- net D-: track 0.00 -> 41.6 mm, vias 0 -> 2
- net GNDPWR: track 0.00 -> 33.7 mm
- net C4: track 0.00 -> 33.2 mm, vias 0 -> 2
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- added copper zone on B.Cu, net GND
- added copper zone on F.Cu, net GND
- removed copper zone on F.Cu, net (none)
Other:
- board outline added: 99.5 x 63 mm
- board text added: "3V3"
- board text added: "5V"
- board text added: "BOOT0"
- board text added: "GND"
- board text added: "GPNGR"
- board text added: "Knobert V 0.01"
- board text added: "NRST"
- board text added: "SCL"
- board text added: "SDA"
- board text added: "SWCLK"
- board text added: "SWDIO"
- board text removed: "EXAMPLE COPPER POUR"
