File: kicad_files/ledmatrix.kicad_sch (KiCad schematic)
At the start: 36 parts

Commit message: Added oled
Parts:
- renumbered D13 to D27, D13 to D28, D13 to D29, D13 to D30, D13 to D31, D13 to D32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

Commit message: beta pcb layout
Parts:
- C1: footprint acheron_Components:C_0402_1005Metric -> Capacitor_SMD:C_0805_2012Metric
- R7: footprint acheron_Components:R_0402_1005Metric -> Resistor_SMD:R_0805_2012Metric
- renumbered D27 to D14, D31 to D15, D35 to D16, D28 to D17, D32 to D18, D36 to D19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
