File: kicad_files/mcu.kicad_sch (KiCad schematic)
At the start: 12 parts, among them J1 ARM JTAG, U1 STM32F072-LQFP48

Commit message: beta pcb layout
Parts:
- C1: renamed from C10; footprint acheron_Components:C_0402_1005Metric -> Capacitor_SMD:C_0805_2012Metric
- C2: renamed from C9; footprint acheron_Components:C_0402_1005Metric -> Capacitor_SMD:C_0805_2012Metric
- C3: renamed from C2; footprint acheron_Components:C_0402_1005Metric -> Capacitor_SMD:C_0805_2012Metric
- C4: renamed from C1; footprint acheron_Components:C_0402_1005Metric -> Capacitor_SMD:C_0805_2012Metric
- C5, C6: footprint acheron_Components:C_0402_1005Metric -> Capacitor_SMD:C_0805_2012Metric
- C7: renamed from C3; footprint acheron_Components:C_0402_1005Metric -> Capacitor_SMD:C_0805_2012Metric
- C8: renamed from C4; footprint acheron_Components:C_0402_1005Metric -> Capacitor_SMD:C_0805_2012Metric
- R1, R2: footprint acheron_Components:R_0402_1005Metric -> Resistor_SMD:R_0805_2012Metric
Connections:
- net C0: now also U1.18 (PB0/TIM3_CH3/ADC_IN8)
- net C1: now also U1.19 (PB1/TIM3_CH4/TIM14_CH1/ADC_IN9)
- net C2: now also U1.45 (I2C1_SCL/TIM16_CH1/PB8)
- net C3: now also U1.46 (SPI2_NSS/I2S2_WS/I2C1_SDA/TIM17_CH1/PB9)
- net C4: now also U1.5 (PF0/OSC_IN)
- net R0: now also U1.17 (PA7/TIM3_CH2/TIM14_CH1/ADC_IN7)
- net R1: now also U1.30 (TIM1_CH2/PA9)
- net R2: now also U1.31 (TIM1_CH3/PA10)
Changed lines of the file:
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@@
     )
   )
-  (global_label "C0" (shape output) (at 52.07 159.385 90) (fields_autoplaced)
-    (effects (font (size 1 1)) (justify left))
-    (property "Intersheetrefs" "${INTERSHEET_REFS}" (at 52.07 155.0697 90)
-      (effects (font (size 1.27 1.27)) (justify left) hide)
-    )
-  )
-  (global_label "R1" (shape input) (at 74.295 156.21 180) (fields_autoplaced)
+  (global_label "C0" (shape output) (at 88.9 139.7 270) (fields_autoplaced)
     (effects (font (size 1 1)) (justify right))
-    (property "Intersheetrefs" "${INTERSHEET_REFS}" (at 69.9797 156.21 0)
+    (property "Intersheetrefs" "${INTERSHEET_REFS}" (at 88.9 144.0153 90)
       (effects (font (size 1.27 1.27)) (justify right) hide)
     )
   )
-  (global_label "C3" (shape output) (at 61.595 159.385 90) (fields_autoplaced)
-    (effects (font (size 1 1)) (justify left))
-    (property "Intersheetrefs" "${INTERSHEET_REFS}" (at 61.595 155.0697 90)
+  (global_label "R1" (shape input) (at 139.7 96.52 0) (fields_autoplaced)
+    (effects (font (size 1 1)) (justify left))
+    (property "Intersheetrefs" "${INTERSHEET_REFS}" (at 144.0153 96.52 0)
+      (effects (font (size 1.27 1.27)) (justify left) hide)
+    )
+  )
+  (global_label "C3" (shape output) (at 69.85 44.45 90) (fields_autoplaced)
+    (effects (font (size 1 1)) (justify left))
+    (property "Intersheetrefs" "${INTERSHEET_REFS}" (at 69.85 40.1347 90)
       (effects (font (size 1.27 1.27)) (justify left) hide)
     )
@@
     )
   )
-  (global_label "C4" (shape output) (at 64.77 159.385 90) (fields_autoplaced)
-    (effects (font (size 1 1)) (justify left))
-    (property "Intersheetrefs" "${INTERSHEET_REFS}" (at 64.77 155.0697 90)
-      (effects (font (size 1.27 1.27)) (justify left) hide)
+  (global_label "C4" (shape output) (at 44.45 82.55 180) (fields_autoplaced)
+    (effects (font (size 1 1)) (justify right))
+    (property "Intersheetrefs" "${INTERSHEET_REFS}" (at 40.1347 82.55 0)
+      (effects (font (size 1.27 1.27)) (justify right) hide)
     )
   )
@@
     )
   )
-  (global_label "C1" (shape output) (at 55.245 159.385 90) (fields_autoplaced)
-    (effects (font (size 1 1)) (justify left))
-    (property "Intersheetrefs" "${INTERSHEET_REFS}" (at 55.245 155.0697 90)
-      (effects (font (size 1.27 1.27)) (justify left) hide)
+  (global_label "C1" (shape output) (at 95.25 139.7 270) (fields_autoplaced)
+    (effects (font (size 1 1)) (justify right))
+    (property "Intersheetrefs" "${INTERSHEET_REFS}" (at 95.25 144.0153 90)
+      (effects (font (size 1.27 1.27)) (justify right) hide)
     )
   )
@@
     )
   )
-  (global_label "C2" (shape output) (at 58.42 159.385 90) (fields_autoplaced)
-    (effects (font (size 1 1)) (justify left))
-    (property "Intersheetrefs" "${INTERSHEET_REFS}" (at 58.42 155.0697 90)
+  (global_label "C2" (shape output) (at 76.2 44.45 90) (fields_autoplaced)
+    (effects (font (size 1 1)) (justify left))
+    (property "Intersheetrefs" "${INTERSHEET_REFS}" (at 76.2 40.1347 90)
       (effects (font (size 1.27 1.27)) (justify left) hide)
     )
@@
     )
   )
-  (global_label "R0" (shape input) (at 74.295 153.035 180) (fields_autoplaced)
+  (global_label "R0" (shape input) (at 82.55 139.7 270) (fields_autoplaced)
     (effects (font (size 1 1)) (justify right))
-    (property "Intersheetrefs" "${INTERSHEET_REFS}" (at 69.9797 153.035 0)
+    (property "Intersheetrefs" "${INTERSHEET_REFS}" (at 82.55 144.0153 90)
       (effects (font (size 1.27 1.27)) (justify right) hide)
     )
@@
     )
   )
-  (global_label "R2" (shape input) (at 74.295 159.385 180) (fields_autoplaced)
-    (effects (font (size 1 1)) (justify right))
-    (property "Intersheetrefs" "${INTERSHEET_REFS}" (at 69.9797 159.385 0)
-      (effects (font (size 1.27 1.27)) (justify right) hide)
+  (global_label "R2" (shape input) (at 139.7 90.17 0) (fields_autoplaced)
+    (effects (font (size 1 1)) (justify left))
+    (property "Intersheetrefs" "${INTERSHEET_REFS}" (at 144.0153 90.17 0)
+      (effects (font (size 1.27 1.27)) (justify left) hide)
     )
   )
@@
       (effects (font (size 1 1)) (justify right))
     )
-    (property "Footprint" "acheron_Components:C_0402_1005Metric" (at 123.825 139.7 0)
+    (property "Footprint" "Capacitor_SMD:C_0805_2012Metric" (at 123.825 139.7 0)
       (effects (font (size 1.27 1.27)) hide)
     )
@@
   (symbol (lib_id "Device:C_Small") (at 60.325 41.91 90) (unit 1)
     (in_bom yes) (on_board yes) (dnp no)
-    (property "Reference" "C1" (at 60.3313 36.83 90)
+    (property "Reference" "C4" (at 60.3313 36.83 90)
       (effects (font (size 1 1)))
     )
@@
       (effects (font (size 1 1)))
     )
-    (property "Footprint" "acheron_Components:C_0402_1005Metric" (at 60.325 41.91 0)
+    (property "Footprint" "Capacitor_SMD:C_0805_2012Metric" (at 60.325 41.91 0)
       (effects (font (size 1.27 1.27)) hide)
     )
@@
       (project "Knobert_MacroPad"
         (path "/9ce6b20d-0a6c-402a-b232-5eafd6242eb3/004d1107-75d6-4f15-a7c8-8fef3fe432ed"
-          (reference "C1") (unit 1)
+          (reference "C4") (unit 1)
         )
       )
@@
   (symbol (lib_id "Device:C_Small") (at 139.7 61.595 180) (unit 1)
     (in_bom yes) (on_board yes) (dnp no)
-    (property "Reference" "C3" (at 139.7 53.34 0)
+    (property "Reference" "C7" (at 139.7 53.34 0)
       (effects (font (size 1 1)))
     )
@@
       (effects (font (size 1 1)))
     )
-    (property "Footprint" "acheron_Components:C_0402_1005Metric" (at 139.7 61.595 0)
+    (property "Footprint" "Capacitor_SMD:C_0805_2012Metric" (at 139.7 61.595 0)
       (effects (font (size 1.27 1.27)) hide)
     )
@@
       (project "Knobert_MacroPad"
         (path "/9ce6b20d-0a6c-402a-b232-5eafd6242eb3/004d1107-75d6-4f15-a7c8-8fef3fe432ed"
-          (reference "C3") (unit 1)
+          (reference "C7") (unit 1)
         )
       )
@@
   (symbol (lib_id "Device:C_Small") (at 46.355 50.8 0) (unit 1)
     (in_bom yes) (on_board yes) (dnp no)
-    (property "Reference" "C2" (at 43.815 48.26 0)
+    (property "Reference" "C3" (at 43.815 48.26 0)
       (effects (font (size 1 1)) (justify right))
     )
@@
       (effects (font (size 1 1)) (justify right))
     )
-    (property "Footprint" "acheron_Components:C_0402_1005Metric" (at 46.355 50.8 0)
+    (property "Footprint" "Capacitor_SMD:C_0805_2012Metric" (at 46.355 50.8 0)
       (effects (font (size 1.27 1.27)) hide)
     )
@@
       (project "Knobert_MacroPad"
         (path "/9ce6b20d-0a6c-402a-b232-5eafd6242eb3/004d1107-75d6-4f15-a7c8-8fef3fe432ed"
-          (reference "C2") (unit 1)
+          (reference "C3") (unit 1)
         )
       )
@@
   (symbol (lib_id "Device:C_Small") (at 149.225 61.595 180) (unit 1)
     (in_bom yes) (on_board yes) (dnp no)
-    (property "Reference" "C4" (at 149.225 53.34 0)
+    (property "Reference" "C8" (at 149.225 53.34 0)
       (effects (font (size 1 1)))
     )
@@
       (effects (font (size 1 1)))
     )
-    (property "Footprint" "acheron_Components:C_0402_1005Metric" (at 149.225 61.595 0)
+    (property "Footprint" "Capacitor_SMD:C_0805_2012Metric" (at 149.225 61.595 0)
       (effects (font (size 1.27 1.27)) hide)
     )
@@
       (project "Knobert_MacroPad"
         (path "/9ce6b20d-0a6c-402a-b232-5eafd6242eb3/004d1107-75d6-4f15-a7c8-8fef3fe432ed"
-          (reference "C4") (unit 1)
+          (reference "C8") (unit 1)
         )
       )
@@
       (effects (font (size 1 1)) (justify right))
     )
-    (property "Footprint" "acheron_Components:C_0402_1005Metric" (at 123.825 148.59 0)
+    (property "Footprint" "Capacitor_SMD:C_0805_2012Metric" (at 123.825 148.59 0)
       (effects (font (size 1.27 1.27)) hide)
     )
@@
       (effects (font (size 1 1)) (justify left))
     )
-    (property "Footprint" "acheron_Components:R_0402_1005Metric" (at 97.79 36.83 0)
+    (property "Footprint" "Resistor_SMD:R_0805_2012Metric" (at 97.79 36.83 0)
       (effects (font (size 1.27 1.27)) hide)
     )
@@
       (effects (font (size 1 1)) (justify left))
     )
-    (property "Footprint" "acheron_Components:R_0402_1005Metric" (at 91.44 36.83 0)
+    (property "Footprint" "Resistor_SMD:R_0805_2012Metric" (at 91.44 36.83 0)
       (effects (font (size 1.27 1.27)) hide)
     )
@@
   (symbol (lib_id "Device:C_Small") (at 34.925 104.775 0) (unit 1)
     (in_bom yes) (on_board yes) (dnp no)
-    (property "Reference" "C10" (at 34.925 97.79 0)
+    (property "Reference" "C1" (at 34.925 97.79 0)
       (effects (font (size 1 1)))
     )
@@
       (effects (font (size 1 1)))
     )
-    (property "Footprint" "acheron_Components:C_0402_1005Metric" (at 34.925 104.775 0)
+    (property "Footprint" "Capacitor_SMD:C_0805_2012Metric" (at 34.925 104.775 0)
       (effects (font (size 1.27 1.27)) hide)
     )
@@
       (project "Knobert_MacroPad"
         (path "/9ce6b20d-0a6c-402a-b232-5eafd6242eb3/004d1107-75d6-4f15-a7c8-8fef3fe432ed"
-          (reference "C10") (unit 1)
+          (reference "C1") (unit 1)
         )
       )
@@
   (symbol (lib_id "Device:C_Small") (at 44.45 104.775 0) (unit 1)
     (in_bom yes) (on_board yes) (dnp no)
-    (property "Reference" "C9" (at 44.45 97.79 0)
+    (property "Reference" "C2" (at 44.45 97.79 0)
       (effects (font (size 1 1)))
     )
@@
       (effects (font (size 1 1)))
     )
-    (property "Footprint" "acheron_Components:C_0402_1005Metric" (at 44.45 104.775 0)
+    (property "Footprint" "Capacitor_SMD:C_0805_2012Metric" (at 44.45 104.775 0)
       (effects (font (size 1.27 1.27)) hide)
     )
@@
       (project "Knobert_MacroPad"
         (path "/9ce6b20d-0a6c-402a-b232-5eafd6242eb3/004d1107-75d6-4f15-a7c8-8fef3fe432ed"
-          (reference "C9") (unit 1)
-        )
-      )
+          (reference "C2") (unit 1)
+        )
+      )
