File: kicad_files/switchmatrix.kicad_sch (KiCad schematic)
At the start: 25 parts, among them SW1 Mechanical_Switch, SW10 Mechanical_Switch, SW11 Mechanical_Switch, SW12 Mechanical_Switch, SW2 Mechanical_Switch, SW3 Mechanical_Switch, SW4 Mechanical_Switch, SW5 Mechanical_Switch, SW6 Mechanical_Switch, SW7 Mechanical_Switch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

Commit message: beta pcb layout
Other:
- moved on the sheet: D4
Changed lines of the file:
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@@
+    (stroke (width 0) (type default))
+  )
+  (wire (pts (xy 150.495 47.625) (xy 150.495 127))
     (stroke (width 0) (type default))
   )
@@
     (stroke (width 0) (type default))
   )
-  (wire (pts (xy 141.605 42.545) (xy 141.605 66.675))
-    (stroke (width 0) (type default))
-  )
   (wire (pts (xy 40.005 66.675) (xy 40.005 104.775))
     (stroke (width 0) (type default))
@@
     (stroke (width 0) (type default))
   )
-  (wire (pts (xy 153.035 59.69) (xy 150.495 59.69))
+  (wire (pts (xy 153.035 136.525) (xy 150.495 136.525))
     (stroke (width 0) (type default))
   )
@@
     (stroke (width 0) (type default))
   )
-  (wire (pts (xy 150.495 50.165) (xy 150.495 47.625))
-    (stroke (width 0) (type default))
-  )
   (wire (pts (xy 37.465 123.825) (xy 48.895 123.825))
     (stroke (width 0) (type default))
@@
     (stroke (width 0) (type default))
   )
-  (wire (pts (xy 150.495 55.245) (xy 150.495 59.69))
+  (wire (pts (xy 150.495 132.08) (xy 150.495 136.525))
     (stroke (width 0) (type default))
   )
@@
   )
   (wire (pts (xy 74.295 47.625) (xy 74.295 50.165))
+    (stroke (width 0) (type default))
+  )
+  (wire (pts (xy 141.605 42.545) (xy 141.605 143.51))
     (stroke (width 0) (type default))
   )
@@
     (effects (font (size 2 2) (thickness 1.524) bold) (justify left bottom))
   )
-  (global_label "ENCODER_SW2" (shape input) (at 141.605 66.675 0) (fields_autoplaced)
+  (global_label "ENCODER_SW2" (shape input) (at 141.605 143.51 0) (fields_autoplaced)
     (effects (font (size 1 1)) (justify left))
-    (property "Intersheetrefs" "${INTERSHEET_REFS}" (at 154.6823 66.675 0)
+    (property "Intersheetrefs" "${INTERSHEET_REFS}" (at 154.6823 143.51 0)
       (effects (font (size 1.27 1.27)) (justify left) hide)
     )
@@
     )
   )
-  (global_label "ENCODER_SW1" (shape input) (at 153.035 59.69 0) (fields_autoplaced)
+  (global_label "ENCODER_SW1" (shape input) (at 153.035 136.525 0) (fields_autoplaced)
     (effects (font (size 1 1)) (justify left))
-    (property "Intersheetrefs" "${INTERSHEET_REFS}" (at 166.1123 59.69 0)
+    (property "Intersheetrefs" "${INTERSHEET_REFS}" (at 166.1123 136.525 0)
       (effects (font (size 1.27 1.27)) (justify left) hide)
     )
@@
       (project "Knobert_MacroPad"
         (path "/9ce6b20d-0a6c-402a-b232-5eafd6242eb3/f615437f-133a-4080-aefa-693736a8a6cf"
-          (reference "SW8") (unit 1)
+          (reference "SW5") (unit 1)
         )
       )
@@
       (project "Knobert_MacroPad"
         (path "/9ce6b20d-0a6c-402a-b232-5eafd6242eb3/f615437f-133a-4080-aefa-693736a8a6cf"
-          (reference "SW5") (unit 1)
+          (reference "SW7") (unit 1)
         )
       )
@@
       (project "Knobert_MacroPad"
         (path "/9ce6b20d-0a6c-402a-b232-5eafd6242eb3/f615437f-133a-4080-aefa-693736a8a6cf"
-          (reference "SW13") (unit 1)
+          (reference "SW9") (unit 1)
         )
       )
@@
       (project "Knobert_MacroPad"
         (path "/9ce6b20d-0a6c-402a-b232-5eafd6242eb3/f615437f-133a-4080-aefa-693736a8a6cf"
-          (reference "SW14") (unit 1)
+          (reference "SW12") (unit 1)
         )
       )
@@
       (project "Knobert_MacroPad"
         (path "/9ce6b20d-0a6c-402a-b232-5eafd6242eb3/f615437f-133a-4080-aefa-693736a8a6cf"
-          (reference "SW9") (unit 1)
+          (reference "SW8") (unit 1)
         )
       )
@@
       (project "Knobert_MacroPad"
         (path "/9ce6b20d-0a6c-402a-b232-5eafd6242eb3/f615437f-133a-4080-aefa-693736a8a6cf"
-          (reference "SW6") (unit 1)
+          (reference "SW10") (unit 1)
         )
       )
@@
       (project "Knobert_MacroPad"
         (path "/9ce6b20d-0a6c-402a-b232-5eafd6242eb3/f615437f-133a-4080-aefa-693736a8a6cf"
-          (reference "SW7") (unit 1)
+          (reference "SW2") (unit 1)
         )
       )
@@
       (project "Knobert_MacroPad"
         (path "/9ce6b20d-0a6c-402a-b232-5eafd6242eb3/f615437f-133a-4080-aefa-693736a8a6cf"
-          (reference "SW12") (unit 1)
+          (reference "SW6") (unit 1)
         )
       )
@@
       (project "Knobert_MacroPad"
         (path "/9ce6b20d-0a6c-402a-b232-5eafd6242eb3/f615437f-133a-4080-aefa-693736a8a6cf"
-          (reference "D9") (unit 1)
-        )
-      )
-    )
-  )
-  (symbol (lib_id "Device:D_Small") (at 150.495 52.705 270) (unit 1)
+          (reference "D8") (unit 1)
+        )
+      )
+    )
+  )
+  (symbol (lib_id "Device:D_Small") (at 150.495 129.54 270) (unit 1)
     (in_bom yes) (on_board yes) (dnp no) (fields_autoplaced)
-    (property "Reference" "D4" (at 153.035 52.07 90)
-      (effects (font (size 1.27 1.27)) (justify left))
-    )
-    (property "Value" "1N4148W" (at 153.035 54.61 90)
-      (effects (font (size 1.27 1.27)) (justify left))
-    )
-    (property "Footprint" "acheron_Components:D_SOD-123" (at 150.495 52.705 90)
-      (effects (font (size 1.27 1.27)) hide)
-    )
-    (property "Datasheet" "~" (at 150.495 52.705 90)
-      (effects (font (size 1.27 1.27)) hide)
-    )
-    (property "Package" "SOD-123" (at 150.495 52.705 0)
-      (effects (font (size 1.27 1.27)) hide)
-    )
-    (property "Manufacturer" "" (at 150.495 52.705 0)
-      (effects (font (size 1.27 1.27)) hide)
-    )
-    (property "Manufacturer Part Number" "" (at 150.495 52.705 0)
-      (effects (font (size 1.27 1.27)) hide)
-    )
-    (property "Vendor Part Number" "" (at 150.495 52.705 0)
-      (effects (font (size 1.27 1.27)) hide)
-    )
-    (property "Description" "small switching diode" (at 150.495 52.705 0)
+    (property "Reference" "D4" (at 153.035 128.905 90)
+      (effects (font (size 1.27 1.27)) (justify left))
+    )
+    (property "Value" "1N4148W" (at 153.035 131.445 90)
+      (effects (font (size 1.27 1.27)) (justify left))
+    )
+    (property "Footprint" "acheron_Components:D_SOD-123" (at 150.495 129.54 90)
+      (effects (font (size 1.27 1.27)) hide)
+    )
+    (property "Datasheet" "~" (at 150.495 129.54 90)
+      (effects (font (size 1.27 1.27)) hide)
+    )
+    (property "Package" "SOD-123" (at 150.495 129.54 0)
+      (effects (font (size 1.27 1.27)) hide)
+    )
+    (property "Manufacturer" "" (at 150.495 129.54 0)
+      (effects (font (size 1.27 1.27)) hide)
+    )
+    (property "Manufacturer Part Number" "" (at 150.495 129.54 0)
+      (effects (font (size 1.27 1.27)) hide)
+    )
+    (property "Vendor Part Number" "" (at 150.495 129.54 0)
+      (effects (font (size 1.27 1.27)) hide)
+    )
+    (property "Description" "small switching diode" (at 150.495 129.54 0)
       (effects (font (size 1.27 1.27)) hide)
     )
@@
       (project "Knobert_MacroPad"
         (path "/9ce6b20d-0a6c-402a-b232-5eafd6242eb3/f615437f-133a-4080-aefa-693736a8a6cf"
-          (reference "D15") (unit 1)
+          (reference "D13") (unit 1)
         )
       )
@@
       (project "Knobert_MacroPad"
         (path "/9ce6b20d-0a6c-402a-b232-5eafd6242eb3/f615437f-133a-4080-aefa-693736a8a6cf"
-          (reference "SW11") (unit 1)
+          (reference "SW3") (unit 1)
         )
       )
@@
       (project "Knobert_MacroPad"
         (path "/9ce6b20d-0a6c-402a-b232-5eafd6242eb3/f615437f-133a-4080-aefa-693736a8a6cf"
-          (reference "D12") (unit 1)
+          (reference "D6") (unit 1)
         )
       )
@@
       (project "Knobert_MacroPad"
         (path "/9ce6b20d-0a6c-402a-b232-5eafd6242eb3/f615437f-133a-4080-aefa-693736a8a6cf"
-          (reference "D6") (unit 1)
+          (reference "D10") (unit 1)
         )
       )
@@
       (project "Knobert_MacroPad"
         (path "/9ce6b20d-0a6c-402a-b232-5eafd6242eb3/f615437f-133a-4080-aefa-693736a8a6cf"
-          (reference "D11") (unit 1)
+          (reference "D3") (unit 1)
         )
       )
@@
       (project "Knobert_MacroPad"
         (path "/9ce6b20d-0a6c-402a-b232-5eafd6242eb3/f615437f-133a-4080-aefa-693736a8a6cf"
-          (reference "D8") (unit 1)
+          (reference "D5") (unit 1)
         )
       )
@@
       (project "Knobert_MacroPad"
         (path "/9ce6b20d-0a6c-402a-b232-5eafd6242eb3/f615437f-133a-4080-aefa-693736a8a6cf"
-          (reference "D14") (unit 1)
+          (reference "D12") (unit 1)
         )
       )
@@
       (project "Knobert_MacroPad"
         (path "/9ce6b20d-0a6c-402a-b232-5eafd6242eb3/f615437f-133a-4080-aefa-693736a8a6cf"
-          (reference "D10") (unit 1)
+          (reference "D11") (unit 1)
         )
       )
@@
       (project "Knobert_MacroPad"
         (path "/9ce6b20d-0a6c-402a-b232-5eafd6242eb3/f615437f-133a-4080-aefa-693736a8a6cf"
-          (reference "SW10") (unit 1)
+          (reference "SW11") (unit 1)
         )
       )
@@
       (project "Knobert_MacroPad"
         (path "/9ce6b20d-0a6c-402a-b232-5eafd6242eb3/f615437f-133a-4080-aefa-693736a8a6cf"
-          (reference "D3") (unit 1)
+          (reference "D1") (unit 1)
         )
       )
@@
       (project "Knobert_MacroPad"
         (path "/9ce6b20d-0a6c-402a-b232-5eafd6242eb3/f615437f-133a-4080-aefa-693736a8a6cf"
-          (reference "D5") (unit 1)
+          (reference "D7") (unit 1)
         )
       )
@@
       (project "Knobert_MacroPad"
         (path "/9ce6b20d-0a6c-402a-b232-5eafd6242eb3/f615437f-133a-4080-aefa-693736a8a6cf"
-          (reference "D13") (unit 1)
+          (reference "D9") (unit 1)
         )
       )
@@
       (project "Knobert_MacroPad"
         (path "/9ce6b20d-0a6c-402a-b232-5eafd6242eb3/f615437f-133a-4080-aefa-693736a8a6cf"
-          (reference "D7") (unit 1)
+          (reference "D2") (unit 1)
         )
       )
@@
       (project "Knobert_MacroPad"
         (path "/9ce6b20d-0a6c-402a-b232-5eafd6242eb3/f615437f-133a-4080-aefa-693736a8a6cf"
-          (reference "SW3") (unit 1)
-        )
-      )
+          (reference "SW1") (unit 1)
+        )
+      )
